File: kicad/beanbot_312/beanbot_312.kicad_sch (KiCad schematic)
At the start: 70 parts, among them M1 P&O2_VOEDING, M10 P&O2_MEETPUNT, M11 P&O2_ULTRASONE_HC_SR04, M12 P&O2_MEETPUNT, M13 P&O2_MEETPUNT, M14 P&O2_GEWICHTSENSOR, M15 P&O2_MEETPUNT, M16 P&O2_MEETPUNT, M17 P&O2_MEETPUNT, M18 P&O2_MEETPUNT, M19 P&O2_MEETPUNT, M2 P&O2_MEETPUNT, M20 P&O2_KLEURSENSOR, M21 P&O2_MEETPUNT, M22 P&O2_MEETPUNT, M23 P&O2_RESISTOR, M24 P&O2_MEETPUNT, M25 P&O2_RESISTOR, M26 P&O2_RESISTOR, M27 P&O2_MEETPUNT, M28 P&O2_DC-MOTOR, M29 P&O2_RESISTOR, M3 P&O2_RESISTOR, M30 P&O2_MEETPUNT, M31 P&O2_DC-MOTOR, M32 P&O2_MEETPUNT, M33 P&O2_RESISTOR, M34 P&O2_MEETPUNT, M35 P&O2_RESISTOR, M36 P&O2_RESISTOR, M37 P&O2_MEETPUNT, M38 P&O2_DC-MOTOR, M39 P&O2_RESISTOR, M4 P&O2_MEETPUNT, M40 P&O2_MEETPUNT, M41 P&O2_DC-MOTOR, M42 P&O2_MEETPUNT, M43 P&O2_RESISTOR, M44 P&O2_MEETPUNT, M45 P&O2_RESISTOR, M46 P&O2_RESISTOR, M47 P&O2_MEETPUNT, M48 P&O2_DC-MOTOR, M49 P&O2_RESISTOR, M5 P&O2_RGB_LED, M50 P&O2_MEETPUNT, M51 P&O2_DC-MOTOR, M52 P&O2_MEETPUNT, M53 P&O2_MOSFET, M54 P&O2_MOSFET, M55 P&O2_MOSFET, M56 P&O2_MOSFET, M57 P&O2_MOSFET, M58 P&O2_MOSFET, M6 P&O2_RESISTOR, M7 P&O2_MEETPUNT, M8 P&O2_RESISTOR, M9 P&O2_RESISTOR, U1 P&O2_ARDUINO_MEGA, U2 LCD-016N002L

Commit message: Latest changes
Parts:
- removed U2: LCD-016N002L, Display:LCD-016N002L, symbol Display_Character:LCD-016N002L
- gave numbers to parts that had none: 4
Connections:
- net 5V: now also SV1.2; no longer M8.2
- net D1_INM6: now also U1.25 (D5)
- net D_LCDDB4: now also SV1.11
- net D_LCDDB5: now also SV1.12
- net D_LCDDB6: now also SV1.13
- net D_LCDDB7: now also SV1.14
- net D_LCDE: now also SV1.6
- net D_LCDRS: now also SV1.4
- net GND: now also M8.2, SV1.15, SV1.3
- net M2OUT1: no longer U4.14 (4Y)
- net M2OUT2: now also U4.14 (4Y)
- net M4OUT1: no longer M25.1, U3.14 (4Y)
- net at SV1.16: now also M8.1
- new net M4OUT2: M25.1, U3.14 (4Y)
Other:
- note removed: "A1 = LED+ K1 = LED-"
- moved on the sheet: SV1

Commit message: Changed DC to servomotor
Parts:
- removed D1: P&O2_DIODE, 1_P&O2_lib:P&O2_DIODE, symbol 1_P&O2_lib:P&O2_DIODE
- removed M23, M26: P&O2_RESISTOR, 1_P&O2_lib:P&O2_RES, symbol 1_P&O2_lib:P&O2_RESISTOR
- removed M24, M30: P&O2_MEETPUNT, 1_P&O2_lib:P&O2_MEETPUNT, symbol 1_P&O2_lib:P&O2_MEETPUNT
- removed M28: P&O2_DC-MOTOR, 1_P&O2_lib:P&O2_2PIN-SCREW-5.08, symbol 1_P&O2_lib:P&O2_DC-MOTOR
- removed M53: P&O2_MOSFET, 1_P&O2_lib:P&O2_TO220, symbol 1_P&O2_lib:P&O2_MOSFET
- added M? (x2): P&O2_MEETPUNT, 1_P&O2_lib:P&O2_MEETPUNT, symbol 1_P&O2_lib:P&O2_MEETPUNT
- added M?: P&O2_SERVOMOTOR, P&O2_lib_SERVO-3PIN, symbol 1_P&O2_lib:P&O2_SERVOMOTOR
Connections:
- net 12V: now also M?.2 (VCC)
- net GND: now also M?.1 (GND), M?.1 (TP)
- net PWM_LEDB: no longer U1.30 (D11)
- net PWM_LEDG: no longer U1.24 (D12)
- net PWM_LEDR: no longer U1.22 (D13)
- net A_LEDB: now reaches U1.5 (A2)
- net A_LEDR: now reaches U1.6 (A3)
- net A_LEDG: now reaches U1.7 (A4)
- new net PWM_S1: M?.1 (TP), M?.3 (SIGN), U1.22 (D13)

Commit message: Latest changes
Parts:
- gave numbers to parts that had none: 3
Changed lines of the file:
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@@
   (symbol (lib_id "1_P&O2_lib:P&O2_MEETPUNT") (at 299.72 96.52 90) (unit 1)
     (in_bom yes) (on_board yes) (fields_autoplaced)
-    (property "Reference" "M?" (id 0) (at 303.53 85.8668 90)
+    (property "Reference" "M26" (id 0) (at 303.53 85.8668 90)
       (effects (font (size 1.143 1.143)) (justify right))
     )
@@
   (symbol (lib_id "1_P&O2_lib:P&O2_SERVOMOTOR") (at 276.86 96.52 270) (unit 1)
     (in_bom yes) (on_board yes) (fields_autoplaced)
-    (property "Reference" "M?" (id 0) (at 276.86 96.52 0)
+    (property "Reference" "M24" (id 0) (at 276.86 96.52 0)
       (effects (font (size 1.143 1.143)) hide)
     )
@@
   (symbol (lib_id "1_P&O2_lib:P&O2_MEETPUNT") (at 25.4 270.51 0) (unit 1)
     (in_bom yes) (on_board yes) (fields_autoplaced)
-    (property "Reference" "M?" (id 0) (at 36.0532 275.59 0)
+    (property "Reference" "M23" (id 0) (at 36.0532 275.59 0)
       (effects (font (size 1.143 1.143)))
     )
@@
       (reference "M22") (unit 1) (value "P&O2_MEETPUNT") (footprint "1_P&O2_lib:P&O2_MEETPUNT")
     )
+    (path "/e4f0c1be-6cfe-44fa-97aa-f7846df8f231"
+      (reference "M23") (unit 1) (value "P&O2_MEETPUNT") (footprint "1_P&O2_lib:P&O2_MEETPUNT")
+    )
+    (path "/b5e46137-190b-4f90-8a4b-0c73a1112167"
+      (reference "M24") (unit 1) (value "P&O2_SERVOMOTOR") (footprint "P&O2_lib_SERVO-3PIN")
+    )
     (path "/cbfd7726-f525-49e8-bccc-7ee91e69e7e6"
       (reference "M25") (unit 1) (value "P&O2_RESISTOR") (footprint "1_P&O2_lib:P&O2_RES")
     )
+    (path "/733340a5-e748-4578-bc19-cbac72592315"
+      (reference "M26") (unit 1) (value "P&O2_MEETPUNT") (footprint "1_P&O2_lib:P&O2_MEETPUNT")
+    )
     (path "/bd109386-669e-493f-a0af-f6eef7558c5c"
       (reference "M27") (unit 1) (value "P&O2_MEETPUNT") (footprint "1_P&O2_lib:P&O2_MEETPUNT")
@@
       (reference "M58") (unit 1) (value "P&O2_MOSFET") (footprint "1_P&O2_lib:P&O2_TO220")
     )
-    (path "/733340a5-e748-4578-bc19-cbac72592315"
-      (reference "M?") (unit 1) (value "P&O2_MEETPUNT") (footprint "1_P&O2_lib:P&O2_MEETPUNT")
-    )
-    (path "/b5e46137-190b-4f90-8a4b-0c73a1112167"
-      (reference "M?") (unit 1) (value "P&O2_SERVOMOTOR") (footprint "P&O2_lib_SERVO-3PIN")
-    )
-    (path "/e4f0c1be-6cfe-44fa-97aa-f7846df8f231"
-      (reference "M?") (unit 1) (value "P&O2_MEETPUNT") (footprint "1_P&O2_lib:P&O2_MEETPUNT")
-    )
     (path "/31e61e3b-86e2-42f7-90c4-159698048ccb"
