File: kicad/beanbot_312/beanbot_312.kicad_pcb (KiCad board)
At the start: 2 copper layers, 0 parts

Commit message: First attempt for DC motor & tweaked scheme a little
Parts:
- added M1: P&O2_MEETPUNT, 1_P&O2_lib:P&O2_MEETPUNT, F.Cu at (-94.5, 152.9)
- added M10: P&O2_RGB_LED, 1_P&O2_lib:P&O2_RGB_LED, F.Cu at (-180.0, 196.9)
- added M11: P&O2_RESISTOR, 1_P&O2_lib:P&O2_RESISTOR, F.Cu at (-235.7, 144.9)
- added M12: P&O2_MEETPUNT, 1_P&O2_lib:P&O2_MEETPUNT, F.Cu at (-36.5, 158.9)
- added M13: P&O2_RESISTOR, 1_P&O2_lib:P&O2_RESISTOR, F.Cu at (-205.7, 106.9)
- added M14: P&O2_MOSFET, 1_P&O2_lib:P&O2_TO220, F.Cu at (-111.0, 129.9)
- added M15: P&O2_RESISTOR, 1_P&O2_lib:P&O2_RESISTOR, F.Cu at (-204.7, 91.9)
- added M16: P&O2_ULTRASONE_HC_SR04, 1_P&O2_lib:P&O2_ULTRASONE, F.Cu at (-202.7, 125.9)
- added M17: P&O2_MEETPUNT, 1_P&O2_lib:P&O2_MEETPUNT, F.Cu at (-82.5, 181.9)
- added M18: P&O2_MEETPUNT, 1_P&O2_lib:P&O2_MEETPUNT, F.Cu at (-81.5, 192.9)
- added M19: P&O2_MEETPUNT, 1_P&O2_lib:P&O2_MEETPUNT, F.Cu at (-134.7, 153.9)
- added M2: P&O2_MEETPUNT, 1_P&O2_lib:P&O2_MEETPUNT, F.Cu at (-70.7, 169.9)
- added M20: P&O2_MEETPUNT, 1_P&O2_lib:P&O2_MEETPUNT, F.Cu at (-60.7, 192.9)
- added M21: P&O2_GEWICHTSENSOR2, 1_P&O2_lib:P&O2_GEWICHTSENSOR-4PIN, F.Cu at (-100.5, 95.9)
- added M22: P&O2_MEETPUNT, 1_P&O2_lib:P&O2_MEETPUNT, F.Cu at (-110.7, 188.9)
- added M23: P&O2_MEETPUNT, 1_P&O2_lib:P&O2_MEETPUNT, F.Cu at (-104.7, 183.9)
- added M24: P&O2_MEETPUNT, 1_P&O2_lib:P&O2_MEETPUNT, F.Cu at (-139.0, 184.9)
- added M25: P&O2_KLEURSENSOR, 1_P&O2_lib:P&O2_KLEURENSENSOR-8PIN, F.Cu at (-72.2, 125.2)
- added M26: P&O2_MEETPUNT, 1_P&O2_lib:P&O2_MEETPUNT, F.Cu at (-38.7, 184.9)
- added M27: P&O2_MEETPUNT, 1_P&O2_lib:P&O2_MEETPUNT, F.Cu at (-57.5, 150.9)
- added M28: P&O2_MEETPUNT, 1_P&O2_lib:P&O2_MEETPUNT, F.Cu at (-121.7, 170.9)
- added M29: P&O2_RELAIS-DP, 1_P&O2_lib:P&O2_RELAY-DP, F.Cu at (178.3, 64.6)
- added M3: P&O2_RESISTOR, 1_P&O2_lib:P&O2_RESISTOR, F.Cu at (-235.7, 99.9)
- added M30: P&O2_DC-MOTOR, 1_P&O2_lib:P&O2_2PIN-SCREW-5.08, F.Cu at (193.0, 54.5)
- added M31: P&O2_RELAIS-DP, 1_P&O2_lib:P&O2_RELAY-DP, F.Cu at (-192.7, 40.9)
- added M32: P&O2_DC-MOTOR, 1_P&O2_lib:P&O2_2PIN-SCREW-5.08, F.Cu at (-147.2, 94.9)
- added M33: P&O2_RELAIS-DP, 1_P&O2_lib:P&O2_RELAY-DP, F.Cu at (-237.7, 40.9)
- added M34: P&O2_DC-MOTOR, 1_P&O2_lib:P&O2_2PIN-SCREW-5.08, F.Cu at (-182.0, 137.9)
- added M35: P&O2_DIODE, 1_P&O2_lib:P&O2_DIODE, F.Cu at (180.3, 91.5)
- added M36: P&O2_DIODE, 1_P&O2_lib:P&O2_DIODE, F.Cu at (-198.7, 79.9)
- added M37: P&O2_DIODE, 1_P&O2_lib:P&O2_DIODE, F.Cu at (-180.7, 65.9)
- added M38: P&O2_MEETPUNT, 1_P&O2_lib:P&O2_MEETPUNT, F.Cu at (172.7, 83.0)
- added M39: P&O2_MEETPUNT, 1_P&O2_lib:P&O2_MEETPUNT, F.Cu at (-91.5, 162.9)
- added M4: P&O2_MOSFET, 1_P&O2_lib:P&O2_TO220, F.Cu at (-98.7, 67.9)
- added M40: P&O2_MEETPUNT, 1_P&O2_lib:P&O2_MEETPUNT, F.Cu at (-151.0, 165.9)
- added M41: P&O2_MEETPUNT, 1_P&O2_lib:P&O2_MEETPUNT, F.Cu at (193.4, 73.5)
- added M42: P&O2_MEETPUNT, 1_P&O2_lib:P&O2_MEETPUNT, F.Cu at (-46.7, 123.9)
- added M43: P&O2_MEETPUNT, 1_P&O2_lib:P&O2_MEETPUNT, F.Cu at (-53.7, 160.3)
- added M44: P&O2_RESISTOR, 1_P&O2_lib:P&O2_RESISTOR, F.Cu at (193.4, 88.5)
- added M45: P&O2_RESISTOR, 1_P&O2_lib:P&O2_RESISTOR, F.Cu at (-236.7, 112.9)
- added M46: P&O2_RESISTOR, 1_P&O2_lib:P&O2_RESISTOR, F.Cu at (-148.7, 40.9)
- added M47: P&O2_MOSFET, 1_P&O2_lib:P&O2_TO220, F.Cu at (190.9, 67.0)
- added M48: P&O2_MOSFET, 1_P&O2_lib:P&O2_TO220, F.Cu at (-179.0, 165.9)
- added M49: P&O2_MOSFET, 1_P&O2_lib:P&O2_TO220, F.Cu at (-167.0, 141.9)
- added M5: P&O2_RESISTOR, 1_P&O2_lib:P&O2_RESISTOR, F.Cu at (-111.7, 42.9)
- added M50: P&O2_MEETPUNT, 1_P&O2_lib:P&O2_MEETPUNT, F.Cu at (180.7, 83.0)
- added M51: P&O2_MEETPUNT, 1_P&O2_lib:P&O2_MEETPUNT, F.Cu at (-56.7, 182.9)
- added M52: P&O2_MEETPUNT, 1_P&O2_lib:P&O2_MEETPUNT, F.Cu at (-96.7, 192.9)
- added M6: P&O2_MEETPUNT, 1_P&O2_lib:P&O2_MEETPUNT, F.Cu at (-77.5, 146.9)
- added M7: P&O2_RESISTOR, 1_P&O2_lib:P&O2_RESISTOR, F.Cu at (-237.7, 162.9)
- added M8: P&O2_MOSFET, 1_P&O2_lib:P&O2_TO220, F.Cu at (-137.0, 116.9)
- added M9: P&O2_RESISTOR, 1_P&O2_lib:P&O2_RESISTOR, F.Cu at (-236.7, 127.9)
Routing:
- net Net-(M29-Pad14): track 0.00 -> 73.3 mm
- net /12V: track 0.00 -> 44.5 mm
- net Net-(M29-Pad21): track 0.00 -> 23.5 mm
- net Net-(M29-Pad11): track 0.00 -> 11.0 mm
- net /PWM_M3: track 0.00 -> 8.76 mm
- net /D_RELM3: track 0.00 -> 5.77 mm
Other:
- board outline added: 384.6 x 100.4 mm

Commit message: Almost finished
Parts:
- removed M22: P&O2_MEETPUNT, 1_P&O2_lib:P&O2_MEETPUNT
- moved M33 422.2 mm to (179.4, 106.3)
- moved M45 384.4 mm to (142.8, 51.7), turned to 180 degrees
- moved M11 373.3 mm to (136.0, 111.0)
- moved M34 371.9 mm to (189.6, 121.8)
- moved M7 364.9 mm to (118.2, 82.8), turned to 90 degrees
- moved M36 363.3 mm to (164.2, 64.7), turned to -90 degrees
- moved M48 362.5 mm to (164.2, 49.1)
- moved M3 354.0 mm to (118.2, 106.3), turned to 90 degrees
- moved M9 351.9 mm to (112.2, 82.8), turned to 90 degrees
- moved M16 336.6 mm to (132.7, 98.5)
- moved M37 335.9 mm to (152.4, 108.8), turned to 90 degrees
- moved M46 333.1 mm to (174.4, 121.8)
- moved M31 331.2 mm to (137.4, 67.1), turned to 180 degrees
- moved M13 327.5 mm to (118.2, 59.1), turned to 90 degrees
- moved M49 319.9 mm to (152.4, 124.3), turned to 180 degrees
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Routing:
- net /12V: track 44.5 -> 169.1 mm
- net /5V: track 0.00 -> 116.6 mm
- net Net-(M33-Pad14): track 0.00 -> 74.0 mm
- net Net-(M31-Pad14): track 0.00 -> 73.6 mm
- net Net-(M33-Pad21): track 0.00 -> 27.3 mm
- net Net-(M31-Pad21): track 0.00 -> 25.9 mm
- net Net-(M10-Pad4): track 0.00 -> 24.4 mm
- net /PWM_LEDG: track 0.00 -> 23.2 mm
- net /PWM_LEDB: track 0.00 -> 22.1 mm
- net /PWM_LEDR: track 0.00 -> 21.6 mm
- net Net-(M10-Pad1): track 0.00 -> 21.0 mm
- net Net-(M33-Pad11): track 0.00 -> 11.8 mm
- net Net-(M31-Pad11): track 0.00 -> 11.3 mm
- net Net-(M4-Pad2): track 0.00 -> 10.4 mm
- net /PWM_M1: track 0.00 -> 9.30 mm
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- added copper zone on B.Cu, net /GND
Other:
- board size 384.6 x 100.4 mm -> 100 x 84 mm
- board text added: "Bean Bot Team 312 R.M. L.M. H.M. M.M. J.N. R.N. M.S. I.V."

Commit message: Fix warnings
Parts:
- moved M4 1.25 mm to (103.7, 107.2)
- moved M37 0.10 mm to (152.5, 108.8)
Routing:
- net /PWM_LEDR: track 21.6 -> 20.3 mm
- net Net-(M4-Pad2): track 10.4 -> 11.6 mm
