File: kicad/beanbot_312/beanbot_312.kicad_pcb (KiCad board)
At the start: 2 copper layers, 100 x 100 mm, 45 parts, among them M1 >VALUE, M10 >VALUE, M11 >VALUE, M12 >VALUE, M13 >VALUE, M14 P&O2_MOSFET, M15 >VALUE, M16 P&O2_ULTRASONE_HC_SR04, M17 >VALUE, M18 >VALUE, M19 >VALUE, M2 >VALUE, M20 >VALUE, M21 P&O2_GEWICHTSENSOR2, M23 >VALUE, M24 >VALUE, M25 P&O2_KLEURSENSOR, M26 >VALUE, M27 >VALUE, M28 >VALUE, M29 P&O2_RELAIS-DP, M3 >VALUE, M30 P&O2_DC-MOTOR, M31 P&O2_RELAIS-DP, M32 P&O2_DC-MOTOR, M35 >VALUE, M36 >VALUE, M38 >VALUE, M39 >VALUE, M4 P&O2_MOSFET, M41 >VALUE, M42 >VALUE, M44 >VALUE, M45 >VALUE, M47 P&O2_MOSFET, M48 P&O2_MOSFET, M5 >VALUE, M50 >VALUE, M51 >VALUE, M6 >VALUE, M7 >VALUE, M8 P&O2_MOSFET, M9 >VALUE, U1 P&O2_ARDUINO_MEGA_SHIELD

Commit message: Cleared warnings
Connections:
- U1 pad 2: unconnected-(U1-Pad2) -> /GND
Routing:
- net /12V: track 206.0 -> 213.6 mm
- net /5V: track 218.3 -> 220.9 mm
Changed lines of the file:
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@@
       (net 43 "unconnected-(U1-Pad2)") (pinfunction "GND") (pintype "bidirectional"))
     (pad "2" thru_hole circle (at 3.744999 -1.525001 270) (size 1.55 1.55) (drill 1.04) (layers *.Cu *.Mask)
-      (net 43 "unconnected-(U1-Pad2)") (pinfunction "GND") (pintype "bidirectional"))
+      (net 3 "/GND") (pinfunction "GND") (pintype "bidirectional"))
     (pad "2" thru_hole circle (at 33.234409 -46.076605 270) (size 1.55 1.55) (drill 1.02) (layers *.Cu *.Mask)
       (net 43 "unconnected-(U1-Pad2)") (pinfunction "GND") (pintype "bidirectional"))
@@
       (net 43 "unconnected-(U1-Pad2)") (pinfunction "GND") (pintype "bidirectional"))
     (pad "2" thru_hole circle (at 1.204999 -1.525001 270) (size 1.55 1.55) (drill 1.04) (layers *.Cu *.Mask)
-      (net 43 "unconnected-(U1-Pad2)") (pinfunction "GND") (pintype "bidirectional"))
+      (net 3 "/GND") (pinfunction "GND") (pintype "bidirectional"))
     (pad "2" thru_hole circle (at 10.476007 -29.591997 270) (size 1.55 1.55) (drill 1.02) (layers *.Cu *.Mask)
       (net 43 "unconnected-(U1-Pad2)") (pinfunction "GND") (pintype "bidirectional"))
     (pad "2" thru_hole circle (at 1.204999 -4.065001 270) (size 1.55 1.55) (drill 1.04) (layers *.Cu *.Mask)
-      (net 43 "unconnected-(U1-Pad2)") (pinfunction "GND") (pintype "bidirectional"))
+      (net 3 "/GND") (pinfunction "GND") (pintype "bidirectional"))
     (pad "2" thru_hole circle (at 13.016007 -29.591997 270) (size 1.55 1.55) (drill 1.02) (layers *.Cu *.Mask)
       (net 43 "unconnected-(U1-Pad2)") (pinfunction "GND") (pintype "bidirectional"))
@@
       (net 43 "unconnected-(U1-Pad2)") (pinfunction "GND") (pintype "bidirectional"))
     (pad "2" thru_hole circle (at 3.744999 -4.065001 270) (size 1.55 1.55) (drill 1.04) (layers *.Cu *.Mask)
-      (net 43 "unconnected-(U1-Pad2)") (pinfunction "GND") (pintype "bidirectional"))
+      (net 3 "/GND") (pinfunction "GND") (pintype "bidirectional"))
     (pad "3" thru_hole circle (at 22.519981 -0.521544) (size 1.55 1.55) (drill 1.02) (layers *.Cu *.Mask)
       (net 44 "unconnected-(U1-Pad3)") (pinfunction "A0") (pintype "bidirectional"))
@@
   (segment (start 126.724036 80.56) (end 124.888 82.396036) (width 1) (layer "F.Cu") (net 1))
   (segment (start 144.892655 87.992655) (end 133.647345 87.992655) (width 1) (layer "F.Cu") (net 1))
+  (segment (start 142.38561 93.18081) (end 144.92561 93.18081) (width 1) (layer "F.Cu") (net 1))
   (segment (start 142.04 129.64) (end 150 129.64) (width 1) (layer "F.Cu") (net 1))
   (segment (start 150 129.64) (end 171.64 129.64) (width 1) (layer "F.Cu") (net 1))
@@
   (segment (start 140.02542 57.4) (end 134.88192 62.5435) (width 2) (layer "F.Cu") (net 20))
   (segment (start 124.8032 70.1) (end 127.399711 67.503489) (width 2) (layer "F.Cu") (net 20))
+  (segment (start 133.114602 133.947806) (end 133.114602 131.407806) (width 2) (layer "F.Cu") (net 20))
   (segment (start 127.399711 67.503489) (end 129.921931 67.503489) (width 2) (layer "F.Cu") (net 20))
   (segment (start 164.2251 57.4) (end 169.1435 57.4) (width 2) (layer "F.Cu") (net 20))
   (segment (start 174.4435 52.1) (end 177.040011 54.696511) (width 2) (layer "F.Cu") (net 20))
+  (segment (start 135.654602 131.407806) (end 135.654602 133.947806) (width 2) (layer "F.Cu") (net 20))
   (segment (start 186.7 66.90158) (end 181.97714 62.17872) (width 2) (layer "F.Cu") (net 20))
   (segment (start 123.27 133) (end 132.166796 133) (width 2) (layer "F.Cu") (net 20))
@@
   (segment (start 133.114602 133.947806) (end 132.166796 133) (width 2) (layer "F.Cu") (net 20))
   (segment (start 186.7 91.53968) (end 186.7 66.90158) (width 2) (layer "F.Cu") (net 20))
+  (segment (start 133.114602 131.407806) (end 135.654602 131.407806) (width 2) (layer "F.Cu") (net 20))
   (segment (start 177.040011 54.696511) (end 177.040011 57.218731) (width 2) (layer "F.Cu") (net 20))
   (segment (start 164.2251 57.4) (end 140.02542 57.4) (width 2) (layer "F.Cu") (net 20))

Commit message: Backups
Parts:
- added M37: P&O2_RESISTOR, 1_P&O2_lib:P&O2_RESISTOR, F.Cu at (188.0, 74.0)
- added M40: P&O2_RESISTOR, 1_P&O2_lib:P&O2_RESISTOR, F.Cu at (143.0, 56.0)
- added M43: P&O2_MOSFET, 1_P&O2_lib:P&O2_TO220, F.Cu at (196.5, 72.0)
- added M46: P&O2_MOSFET, 1_P&O2_lib:P&O2_TO220, F.Cu at (143.0, 48.2)
- M1, M12, M17, M18, M19, M2, M20, M23, M24, M26, M27, M28, M38, M39, M41, M42, M50, M51, M6: value >VALUE -> P&O2_MEETPUNT
- M10: value >VALUE -> P&O2_RGB_LED
- M11, M13, M15, M3, M44, M45, M5, M7, M9: value >VALUE -> P&O2_RESISTOR
- M35, M36: value >VALUE -> P&O2_DIODE
- moved M45 25.5 mm to (164.0, 65.0), turned to -90 degrees
- moved M44 25.0 mm to (179.0, 90.0), turned to 180 degrees
- moved M36 4.77 mm to (169.0, 63.8)
- moved M35 3.46 mm to (180.3, 95.0)
Connections:
- M29 pad A1: /D_RELM3 -> Net-(M29-PadA1)
- M31 pad A1: /D_RELM2 -> Net-(M31-PadA1)
- U1 pad 39: unconnected-(U1-Pad39) -> /5V
- U1 pad 53: unconnected-(U1-Pad53) -> /5V
Routing:
- net /5V: track 220.9 -> 283.2 mm
- net /D_RELM2: track 31.8 -> 53.6 mm
- net /D_RELM3: track 26.1 -> 46.9 mm
- net Net-(M31-PadA1): track 0.00 -> 14.7 mm
- net Net-(M29-PadA1): track 0.00 -> 14.2 mm
- net /12V: track 213.6 -> 224.1 mm
- net Net-(M31-Pad14): track 77.3 -> 82.2 mm
- net Net-(M29-Pad14): track 86.9 -> 82.8 mm
- net /PWM_M3: track 38.0 -> 41.2 mm
- net /PWM_M2: track 39.0 -> 40.8 mm

Commit message: Edited kicad scheme and pcb
Connections:
- M29 pad A2: /GND -> /5V
- M31 pad A2: /GND -> /5V
Routing:
- net /5V: track 283.2 -> 347.3 mm
Changed lines of the file:
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@@
       (net 72 "Net-(M29-PadA1)") (pinfunction "1") (pintype "passive"))
     (pad "A2" thru_hole circle locked (at -12.5984 -3.87858 90) (size 2.794 2.794) (drill 1.39954) (layers *.Cu *.Paste *.Mask)
-      (net 3 "/GND") (pinfunction "2") (pintype "passive"))
+      (net 1 "/5V") (pinfunction "2") (pintype "passive"))
   )
   (footprint "1_P&O2_lib:P&O2_TO220" (layer "F.Cu")
@@
       (net 73 "Net-(M31-PadA1)") (pinfunction "1") (pintype "passive"))
     (pad "A2" thru_hole circle locked (at -12.5984 -3.87858 180) (size 2.794 2.794) (drill 1.39954) (layers *.Cu *.Paste *.Mask)
-      (net 3 "/GND") (pinfunction "2") (pintype "passive"))
+      (net 1 "/5V") (pinfunction "2") (pintype "passive"))
   )
   (footprint "1_P&O2_lib:P&O2_KLEURENSENSOR-8PIN" (layer "F.Cu")
@@
     (fp_line (start 8.45171 -32.072738) (end 8.45171 -32.072738) (layer "F.SilkS") (width 0.1905))
     (fp_line (start 27.088045 -58.203289) (end 27.088045 -58.965289) (layer "F.SilkS") (width 0.1905))
-    (fp_line (start 28.557631 -51.438393) (end 28.702767 -51.438393) (layer "F.SilkS") (width 0.1905))
     (fp_line (start 28.078621 -26.92741) (end 28.078621 -26.92741) (layer "F.SilkS") (width 0.1905))
     (fp_line (start 29.48941 -44.426603) (end 29.48941 -65.506607) (layer "F.SilkS") (width 0.2))
@@
     (fp_line (start 28.539486 -58.457289) (end 29.011198 -58.457289) (layer "F.SilkS") (width 0.1905))
     (fp_line (start 28.01627 -63.481889) (end 27.834847 -63.481889) (layer "F.SilkS") (width 0.1905))
+    (fp_line (start 28.557631 -51.438393) (end 28.702767 -51.438393) (layer "F.SilkS") (width 0.1905))
     (fp_line (start 28.876927 -29.942745) (end 28.876927 -29.942745) (layer "F.SilkS") (width 0.1905))
     (fp_line (start 35.803871 -35.160625) (end 35.803871 -35.160625) (layer "F.SilkS") (width 0.1905))
@@
     (fp_line (start 37.088398 -25.345344) (end 37.124668 -25.272777) (layer "F.SilkS") (width 0.1905))
     (fp_line (start 33.193021 -5.544306) (end 33.193021 -5.544306) (layer "F.SilkS") (width 0.1875))
+    (fp_line (start 28.949501 -30.124168) (end 28.913214 -30.051601) (layer "F.SilkS") (width 0.1905))
     (fp_line (start 8.107006 -29.739536) (end 8.143294 -29.666969) (layer "F.SilkS") (width 0.1905))
     (fp_line (start 16.57971 -41.909776) (end 16.615998 -41.982345) (layer "F.SilkS") (width 0.1905))
@@
     (fp_line (start 35.455551 -24.692211) (end 35.564415 -24.728496) (layer "F.SilkS") (width 0.1905))
     (fp_line (start 10.844302 -7.363376) (end 11.352302 -8.887378) (layer "F.SilkS") (width 0.254))
+    (fp_line (start 27.91627 -42.281906) (end 27.734846 -42.281906) (layer "F.SilkS") (width 0.1905))
     (fp_line (start 6.771678 -34.987697) (end 6.880542 -34.95141) (layer "F.SilkS") (width 0.1905))
     (fp_line (start 40.482064 -5.777651) (end 40.482064 -5.777651) (layer "F.SilkS") (width 0.1875))
@@
     (fp_line (start 16.518063 -44.678369) (end 16.518063 -44.678369) (layer "F.SilkS") (width 0.1905))
     (fp_line (start 30.326848 -5.758577) (end 30.326848 -5.758577) (layer "F.SilkS") (width 0.1875))
-    (fp_line (start 28.949501 -30.124168) (end 28.913214 -30.051601) (layer "F.SilkS") (width 0.1905))
     (fp_line (start 32.234288 -7.369104) (end 32.234288 -7.369104) (layer "F.SilkS") (width 0.1875))
     (fp_line (start 8.342862 -32.326728) (end 8.342862 -32.326728) (layer "F.SilkS") (width 0.1905))
@@
     (fp_line (start 7.000286 -32.036434) (end 7.000286 -31.92757) (layer "F.SilkS") (width 0.1905))
     (fp_line (start 35.705918 -32.965347) (end 35.742207 -32.892776) (layer "F.SilkS") (width 0.1905))
-    (fp_line (start 27.91627 -42.281906) (end 27.734846 -42.281906) (layer "F.SilkS") (width 0.1905))
     (fp_line (start 35.60912 -50.718185) (end 35.60912 -50.718185) (layer "F.SilkS") (width 0.1905))
     (fp_line (start 35.324909 -55.891889) (end 35.324909 -56.653889) (layer "F.SilkS") (width 0.1905))
@@
   (segment (start 186.85 134.5) (end 194 127.35) (width 1) (layer "F.Cu") (net 1))
   (segment (start 165.144012 76.696202) (end 168 79.55219) (width 1) (layer "F.Cu") (net 1))
+  (segment (start 133.035409 67.624591) (end 133.035409 70.864851) (width 0.5) (layer "F.Cu") (net 1))
   (segment (start 151.95 95.05) (end 144.892655 87.992655) (width 1) (layer "F.Cu") (net 1))
+  (segment (start 150 70.1) (end 138.68 70.1) (width 0.5) (layer "F.Cu") (net 1))
   (segment (start 144.92561 93.18081) (end 150.08081 93.18081) (width 1) (layer "F.Cu") (net 1))
+  (segment (start 161.699253 75.791444) (end 162.604012 76.696202) (width 0.5) (layer "F.Cu") (net 1))
   (segment (start 150 129.64) (end 159.36 129.64) (width 1) (layer "F.Cu") (net 1))
   (segment (start 133.647345 87.992655) (end 136 85.64) (width 1) (layer "F.Cu") (net 1))
   (segment (start 168 79.55219) (end 168 96) (width 1) (layer "F.Cu") (net 1))
   (segment (start 120.82 126.1) (end 120.87 126.05) (width 1) (layer "F.Cu") (net 1))
+  (segment (start 138.68 70.1) (end 134.62 66.04) (width 0.5) (layer "F.Cu") (net 1))
+  (segment (start 133.035409 70.864851) (end 137.962002 75.791444) (width 0.5) (layer "F.Cu") (net 1))
   (segment (start 151.95 95.05) (end 150.08081 93.18081) (width 1) (layer "F.Cu") (net 1))
   (segment (start 128.808 88.04531) (end 128.860655 87.992655) (width 1) (layer "F.Cu") (net 1))
   (segment (start 153 111.5) (end 153 96.1) (width 1) (layer "F.Cu") (net 1))
   (segment (start 165.144012 76.696202) (end 162.604012 76.696202) (width 1) (layer "F.Cu") (net 1))
+  (segment (start 134.62 66.04) (end 133.035409 67.624591) (width 0.5) (layer "F.Cu") (net 1))
   (segment (start 124.888 85.043484) (end 127.889826 88.04531) (width 1) (layer "F.Cu") (net 1))
   (segment (start 159.36 101.073014) (end 159.36 129.64) (width 1) (layer "F.Cu") (net 1))
@@
   (segment (start 114.08 126.1) (end 120.82 126.1) (width 1) (layer "F.Cu") (net 1))
   (segment (start 171.64 129.64) (end 176.5 134.5) (width 1) (layer "F.Cu") (net 1))
+  (segment (start 137.962002 75.791444) (end 161.699253 75.791444) (width 0.5) (layer "F.Cu") (net 1))
   (segment (start 166.196388 97.803612) (end 165.169402 97.803612) (width 1) (layer "F.Cu") (net 1))
+  (segment (start 174.4435 77.2968) (end 165.74461 77.2968) (width 0.5) (layer "B.Cu") (net 1))
   (segment (start 106.51 95.1) (end 140.46642 95.1) (width 1) (layer "B.Cu") (net 1))
+  (segment (start 165.74461 77.2968) (end 165.144012 76.696202) (width 0.5) (layer "B.Cu") (net 1))
   (segment (start 106.24 95.37) (end 106.51 95.1) (width 1) (layer "B.Cu") (net 1))
   (segment (start 140.46642 95.1) (end 142.38561 93.18081) (width 1) (layer "B.Cu") (net 1))
